Commit message: add hardware interface

File: allegro_hand/urdf/allegro_hand_on_stand.urdf.xacro (robot description, xacro)
@@ -4,9 +4,10 @@
   <xacro:arg name="chirality" default="undefined"/>
   <xacro:arg name="prefix" default=""/>
+  <xacro:arg name="real_hardware" default="false"/>
   <!-- ur5 robot -->
   <xacro:include filename="$(find allegro_hand_description)/description/allegro_hand_description.urdf.xacro" />
   <!-- Root link -->
   <link name="world"/>
-  <xacro:allegro_hand chirality="$(arg chirality)" parent="world" prefix="$(arg prefix)" ur5_attachment="true" desk_stand="true">
+  <xacro:allegro_hand chirality="$(arg chirality)" parent="world" real_hardware="$(arg real_hardware)" prefix="$(arg prefix)" ur5_attachment="true" desk_stand="true">
     <origin xyz="0.0 0.0 0" rpy="0.0 0 0.0"/>
   </xacro:allegro_hand>

File: allegro_hand_description/description/allegro_hand_description.urdf.xacro (robot description, xacro)
@@ -551,5 +551,5 @@
         </xacro:unless>
         <!-- ================================ ROS2 CONTROL =============================== -->
-        <xacro:allegro_hand_ros2_control name="${prefix}_allegro_hand_ros2_control" prefix="${prefix}" initial_positions_file="${init_pos_file}" real_hardware="${real_hardware}"/>
+        <xacro:allegro_hand_ros2_control name="allegro_hand" prefix="${prefix}" initial_positions_file="${init_pos_file}" use_real_hardware="${real_hardware}"/>
         <!-- ============================= GAZEBO SIMULATION ============================= -->
         <xacro:unless value="${real_hardware}">

File: allegro_hand_description/description/allegro_hand_ros2_control.xacro (robot description, xacro)
@@ -1,39 +1,60 @@
 <?xml version="1.0"?>
 <robot xmlns:xacro="http://www.ros.org/wiki/xacro">
-    <xacro:macro name="allegro_hand_ros2_control" params="name prefix initial_positions_file real_hardware">
-        <xacro:property name="initial_positions" value="${xacro.load_yaml(initial_positions_file)['initial_positions']}"/>
-        <ros2_control name="${name}" type="system">
-            <xacro:unless value="${real_hardware}">
-              <hardware>
-                <plugin>gz_ros2_control/GazeboSimSystem</plugin>
-              </hardware>
-            </xacro:unless>
-            <xacro:macro name="joint_definition" params="joint_name initial_pos">
-              <joint name="${prefix}_${joint_name}">
-                <command_interface name="effort"/>
-                <state_interface name="effort"/>
-                <state_interface name="position">
-                  <param name="initial_value">${initial_positions[initial_pos]}</param>
-                </state_interface>
-                <state_interface name="velocity"/>
-              </joint>
-            </xacro:macro>
-            <xacro:joint_definition joint_name="joint_00" initial_pos="joint_00" />
-            <xacro:joint_definition joint_name="joint_01" initial_pos="joint_01" />
-            <xacro:joint_definition joint_name="joint_02" initial_pos="joint_02" />
-            <xacro:joint_definition joint_name="joint_03" initial_pos="joint_03" />
-            <xacro:joint_definition joint_name="joint_04" initial_pos="joint_04" />
-            <xacro:joint_definition joint_name="joint_05" initial_pos="joint_05" />
-            <xacro:joint_definition joint_name="joint_06" initial_pos="joint_06" />
-            <xacro:joint_definition joint_name="joint_07" initial_pos="joint_07" />
-            <xacro:joint_definition joint_name="joint_08" initial_pos="joint_08" />
-            <xacro:joint_definition joint_name="joint_09" initial_pos="joint_09" />
-            <xacro:joint_definition joint_name="joint_10" initial_pos="joint_10" />
-            <xacro:joint_definition joint_name="joint_11" initial_pos="joint_11" />
-            <xacro:joint_definition joint_name="joint_12" initial_pos="joint_12" />
-            <xacro:joint_definition joint_name="joint_13" initial_pos="joint_13" />
-            <xacro:joint_definition joint_name="joint_14" initial_pos="joint_14" />
-            <xacro:joint_definition joint_name="joint_15" initial_pos="joint_15" />
-        </ros2_control>
-    </xacro:macro>
+  <xacro:macro name="allegro_hand_ros2_control" params="name prefix initial_positions_file use_real_hardware:=false use_sim_time:=false">
+    <xacro:property name="initial_positions" value="${xacro.load_yaml(initial_positions_file)['initial_positions']}"/>
+    <ros2_control name="${name}" type="system">
+      <!-- ========================================================== -->
+      <!--            SÉLECTION DU PLUGIN HARDWARE                    -->
+      <!-- ========================================================== -->
+      <!-- CAS 1 : ROBOT RÉEL -->
+      <!-- <xacro:if value="${use_real_hardware}"> -->
+      <hardware>
+        <plugin>allegro_hand_interface/AllegroHandHardwareInterface</plugin>
+        <param name="CAN_CH">can0</param>
+        <!-- Ajoutez d'autres paramètres pour votre driver réel ici si nécessaire -->
+      </hardware>
+      <!-- </xacro:if> -->
+      <!-- CAS 2 : SIMULATION GAZEBO -->
+      <!-- <xacro:if value="${use_sim_time and not use_real_hardware}">
+        <hardware>
+          <plugin>gz_ros2_control/GazeboSimSystem</plugin>
+        </hardware>
+      </xacro:if> -->
+      <!-- CAS 3 : VISUALISATION RViz (MOCK) -->
+      <!-- <xacro:unless value="${use_real_hardware or use_sim_time}">
+        <hardware>
+          <plugin>mock_components/GenericSystem</plugin>
+        </hardware>
+      </xacro:unless> -->
+      <!-- ========================================================== -->
+      <!--            DÉFINITION DES ARTICULATIONS                    -->
+      <!-- ========================================================== -->
+      <xacro:macro name="joint_definition" params="joint_name initial_pos">
+        <joint name="${prefix}_${joint_name}">
+          <command_interface name="effort"/>
+          <state_interface name="position">
+            <param name="initial_value">${initial_positions[initial_pos]}</param>
+          </state_interface>
+          <state_interface name="velocity"/>
+        </joint>
+      </xacro:macro>
+      <!-- On appelle la macro pour les 16 articulations -->
+      <xacro:joint_definition joint_name="joint_00" initial_pos="joint_00" />
+      <xacro:joint_definition joint_name="joint_01" initial_pos="joint_01" />
+      <xacro:joint_definition joint_name="joint_02" initial_pos="joint_02" />
+      <xacro:joint_definition joint_name="joint_03" initial_pos="joint_03" />
+      <xacro:joint_definition joint_name="joint_04" initial_pos="joint_04" />
+      <xacro:joint_definition joint_name="joint_05" initial_pos="joint_05" />
+      <xacro:joint_definition joint_name="joint_06" initial_pos="joint_06" />
+      <xacro:joint_definition joint_name="joint_07" initial_pos="joint_07" />
+      <xacro:joint_definition joint_name="joint_08" initial_pos="joint_08" />
+      <xacro:joint_definition joint_name="joint_09" initial_pos="joint_09" />
+      <xacro:joint_definition joint_name="joint_10" initial_pos="joint_10" />
+      <xacro:joint_definition joint_name="joint_11" initial_pos="joint_11" />
+      <xacro:joint_definition joint_name="joint_12" initial_pos="joint_12" />
+      <xacro:joint_definition joint_name="joint_13" initial_pos="joint_13" />
+      <xacro:joint_definition joint_name="joint_14" initial_pos="joint_14" />
+      <xacro:joint_definition joint_name="joint_15" initial_pos="joint_15" />
+    </ros2_control>
+  </xacro:macro>
 </robot>

Commit message: update inertial matrix and readme

File: allegro_hand/urdf/allegro_hand_on_stand.urdf.xacro (robot description, xacro)
@@ -9,5 +9,5 @@
   <!-- Root link -->
   <link name="world"/>
-  <xacro:allegro_hand chirality="$(arg chirality)" parent="world" real_hardware="$(arg real_hardware)" prefix="$(arg prefix)" ur5_attachment="true" desk_stand="true">
+  <xacro:allegro_hand chirality="$(arg chirality)" parent="world" real_hardware="$(arg real_hardware)" prefix="$(arg prefix)" ur5_attachment="true" desk_stand="true" standalone="true">
     <origin xyz="0.0 0.0 0" rpy="0.0 0 0.0"/>
   </xacro:allegro_hand>

File: allegro_hand_description/description/allegro_hand_description.urdf.xacro (robot description, xacro)
@@ -2,5 +2,5 @@
 <robot xmlns:xacro="http://www.ros.org/wiki/xacro" name="allegro_hand">
     <xacro:include filename="$(find allegro_hand_description)/description/allegro_hand_ros2_control.xacro" />
-    <xacro:macro name="allegro_hand" params="chirality parent *origin prefix real_hardware:=false ur5_attachment:=false desk_stand:=false last_links_inertia_factor=1.0">
+    <xacro:macro name="allegro_hand" params="chirality parent *origin prefix real_hardware:=false ur5_attachment:=false desk_stand:=false standalone:=false">
         <!-- ======================== CHIRALITY PARAMS ========================= -->
         <xacro:property name="suffix" value="${chirality}"/>
@@ -75,9 +75,8 @@
             <inertial>
                 <origin xyz="0 0 ${palm_link_z/2}" rpy="0 0 0"/>
-                <mass value="0.4154"/>
-                <inertia
-                    ixx="1e-4" ixy="0.0" ixz="0.0"
-                    iyy="1e-4" iyz="0.0"
-                    izz="1e-4"/>
+                <mass value="4.1685782e-01"/>
+                <inertia ixx="1.3752240e-03" ixy="1.1841496e-05" ixz="-2.7306101e-04"
+                iyx= "1.1841496e-05" iyy="1.2103623e-03" iyz="-2.3172379e-06"
+                izx = "-2.7306101e-04" izy = "-2.3172379e-06" izz="6.2229538e-04"/>
             </inertial>
         </link>
@@ -103,8 +102,8 @@
                 </collision>
                 <inertial>
-                    <mass value="0.0176" />
-                    <origin xyz="0 0 0" rpy="0 0 0"/>
-                    <inertia ixx="1e-5" ixy="0." ixz="0." iyy="1e-5"
-                            iyz="0." izz="1e-5" />
+                    <mass value="7.9809876e-02"/>
+                    <inertia ixx="4.7114004e-05" ixy="-8.5650686e-06" ixz="-5.1403625e-06"
+                    iyx= "-8.5650686e-06" iyy="2.9419559e-05" iyz="-1.2569682e-05"
+                    izx = "-5.1403625e-06" izy = "-1.2569682e-05" izz="4.0511157e-05"/>
                 </inertial>
             </link>
@@ -136,8 +135,8 @@
                 </collision>
                 <inertial>
-                    <mass value="0.0119" />
-                    <origin xyz="0 0 0" rpy="0 0 0"/>
-                    <inertia ixx="1e-5" ixy="0." ixz="0." iyy="1e-5"
-                            iyz="0." izz="1e-5" />
+                    <mass value="1.1350110e-02"/>
+                    <inertia ixx="2.7007029e-06" ixy="3.1772015e-09" ixz="-9.9625696e-09"
+                    iyx= "3.1772015e-09" iyy="2.0578543e-06" iyz="4.1823243e-09"
+                    izx = "-9.9625696e-09" izy = "4.1823243e-09" izz=" 1.2713693e-06"/>
                 </inertial>
             </link>
@@ -168,8 +167,8 @@
                 </collision>
                 <inertial>
-                    <mass value="0.038" />
-                    <origin xyz="0 0 0" rpy="0 0 0"/>
-                    <inertia ixx="1e-5" ixy="0." ixz="0." iyy="1e-5"
-                            iyz="0." izz="1e-5" />
+                    <mass value="4.0206693e-02"/>
+                    <inertia ixx="4.3413941e-06" ixy="9.6355047e-07" ixz="-3.9856829e-07"
+                    iyx= "9.6355047e-07" iyy="2.1797267e-05" iyz="-1.2313988e-08"
+                    izx = "-3.9856829e-07" izy = "-1.2313988e-08" izz="2.0281187e-05"/>
                 </inertial>
             </link>
@@ -200,8 +199,8 @@
                 </collision>
                 <inertial>
-                    <mass value="0.0388" />
-                    <origin xyz="0 0 0" rpy="0 0 0"/>
-                    <inertia ixx="1e-5" ixy="0." ixz="0." iyy="1e-5"
-                                iyz="0." izz="1e-5" />
+                    <mass value=" 4.0750131e-02"/>
+                    <inertia ixx=" 3.9420540e-06" ixy="5.6337647e-07" ixz="-5.3566170e-08"
+                    iyx= "   5.6337647e-07" iyy=" 1.6474691e-05" iyz="-1.8757848e-08"
+                    izx = " -5.3566170e-08" izy = "-1.8757848e-08" izz="1.5477224e-05"/>
                 </inertial>
             </link>
@@ -232,9 +231,9 @@
                 </collision>
                 <inertial>
-                    <mass value="0.0168" />
                     <origin xyz="0 0 0" rpy="0 0 0"/>
-                    <inertia ixx="${last_links_inertia_factor * 9.680e-05}" ixy="0.0" ixz="0.0"
-                            iyy="${last_links_inertia_factor * 9.680e-05}" iyz="0.0"
-                            izz="${last_links_inertia_factor * 9.680e-05}" />
+                    <mass value="1.6654268e-02"/>
+                    <inertia ixx=" 1.4702815e-06" ixy=" 0.0000000e+00" ixz="0.0000000e+00"
+                    iyx= "0.0000000e+00" iyy= " 3.8502616e-06" iyz="0.0000000e+00"
+                    izx = "0.0000000e+00" izy = "0.0000000e+00" izz="3.8502616e-06"/>
                 </inertial>
             </link>
@@ -265,8 +264,8 @@
                 </collision>
                 <inertial>
-                    <mass value="0.0119" />
-                    <origin xyz="0 0 0" rpy="0 0 0"/>
-                    <inertia ixx="1e-5" ixy="0." ixz="0." iyy="1e-5"
-                            iyz="0." izz="1e-5" />
+                    <mass value="1.1350110e-02"/>
+                    <inertia ixx="2.7007029e-06" ixy=" 3.1772169e-09" ixz="-9.9625685e-09"
+                    iyx= " 3.1772169e-09" iyy=" 2.0578543e-06" iyz="4.1823243e-09"
+                    izx = "-9.9625685e-09" izy = " 4.1823243e-09" izz="1.2713693e-06"/>
                 </inertial>
             </link>
@@ -298,8 +297,8 @@
                 </collision>
                 <inertial>
-                    <mass value="0.065" />
-                    <origin xyz="0 0 0" rpy="0 0 0"/>
-                    <inertia ixx="1e-5" ixy="0." ixz="0." iyy="1e-5"
-                            iyz="0." izz="1e-5" />
+                    <mass value="7.1189096e-02"/>
+                    <inertia ixx="7.0483360e-06" ixy=" 2.7238745e-06" ixz="-5.7605847e-07"
+                    iyx= " 2.7238745e-06" iyy=" 7.7935727e-05" iyz="2.1115155e-08"
+                    izx = " -5.7605847e-07" izy = "2.1115155e-08" izz="7.6656552e-05"/>
                 </inertial>
             </link>
@@ -330,8 +329,8 @@
                 </collision>
                 <inertial>
-                    <mass value="0.0355" />
-                    <origin xyz="0 0 0" rpy="0 0 0"/>
-                    <inertia ixx="1e-5" ixy="0." ixz="0." iyy="1e-5"
-                            iyz="0." izz="1e-5" />
+                    <mass value="3.7588606e-02"/>
+                    <inertia ixx="3.8700419e-06" ixy=" 9.4859852e-07" ixz="-3.4727103e-07"
+                    iyx= "  9.4859852e-07" iyy="  2.9392367e-05" iyz=" 4.1019588e-08"
+                    izx = " -3.4727103e-07" izy = " 4.1019588e-08" izz="2.8178175e-05"/>
                 </inertial>
             </link>
@@ -362,8 +361,8 @@
                 </collision>
                 <inertial>
-                    <mass value="0.0096" />
-                    <origin xyz="0 0 0" rpy="0 0 0"/>
-                    <inertia ixx="1e-5" ixy="0." ixz="0." iyy="1e-5"
-                            iyz="0." izz="1e-5" />
+                    <mass value="9.4301124e-03"/>
+                    <inertia ixx=" 1.2117405e-06" ixy="9.9624823e-09" ixz="6.9119137e-10"
+                    iyx= "9.9624823e-09" iyy="2.1794983e-06" iyz="3.1772815e-09"
+                    izx = "6.9119137e-10" izy = "3.1772815e-09" izz="1.5590472e-06"/>
                 </inertial>
             </link>
@@ -394,9 +393,9 @@
                 </collision>
                 <inertial>
-                <mass value="0.0168" />
                     <origin xyz="0 0 0" rpy="0 0 0"/>
-                    <inertia ixx="${last_links_inertia_factor * 9.680e-05}" ixy="0.0" ixz="0.0"
-                            iyy="${last_links_inertia_factor * 9.680e-05}" iyz="0.0"
-                            izz="${last_links_inertia_factor * 9.680e-05}" />
+                    <mass value="1.6654268e-02"/>
+                    <inertia ixx="1.4702815e-06" ixy=" 0.0000000e+00" ixz="0.0000000e+00"
+                    iyx= "0.0000000e+00" iyy= " 3.8502616e-06" iyz="0.0000000e+00"
+                    izx = "0.0000000e+00" izy = "0.0000000e+00" izz="3.8502616e-06"/>
                 </inertial>
             </link>
@@ -553,5 +552,5 @@
         <xacro:allegro_hand_ros2_control name="allegro_hand" prefix="${prefix}" initial_positions_file="${init_pos_file}" use_real_hardware="${real_hardware}"/>
         <!-- ============================= GAZEBO SIMULATION ============================= -->
-        <xacro:unless value="${real_hardware}">
+        <xacro:if value="${standalone}">
             <gazebo>
                 <plugin filename="gz_ros2_control-system" name="gz_ros2_control::GazeboSimROS2ControlPlugin">
@@ -559,5 +558,5 @@
                 </plugin>
             </gazebo>
-        </xacro:unless>
+        </xacro:if>
     </xacro:macro>
 </robot>

File: allegro_hand_description/description/allegro_hand_ros2_control.xacro (robot description, xacro)
@@ -1,25 +1,24 @@
 <?xml version="1.0"?>
 <robot xmlns:xacro="http://www.ros.org/wiki/xacro">
-  <xacro:macro name="allegro_hand_ros2_control" params="name prefix initial_positions_file use_real_hardware:=false use_sim_time:=false">
+  <xacro:macro name="allegro_hand_ros2_control" params="name prefix initial_positions_file use_real_hardware:=false">
     <xacro:property name="initial_positions" value="${xacro.load_yaml(initial_positions_file)['initial_positions']}"/>
     <ros2_control name="${name}" type="system">
       <!-- ========================================================== -->
-      <!--            SÉLECTION DU PLUGIN HARDWARE                    -->
+      <!--                     PLUGIN HARDWARE                        -->
       <!-- ========================================================== -->
-      <!-- CAS 1 : ROBOT RÉEL -->
-      <!-- <xacro:if value="${use_real_hardware}"> -->
-      <hardware>
-        <plugin>allegro_hand_interface/AllegroHandHardwareInterface</plugin>
-        <param name="CAN_CH">can0</param>
-        <!-- Ajoutez d'autres paramètres pour votre driver réel ici si nécessaire -->
-      </hardware>
-      <!-- </xacro:if> -->
-      <!-- CAS 2 : SIMULATION GAZEBO -->
-      <!-- <xacro:if value="${use_sim_time and not use_real_hardware}">
+      <!-- CAS 1 : REEL ROBOT -->
+      <xacro:if value="${use_real_hardware}">
+        <hardware>
+          <plugin>allegro_hand_interface/AllegroHandHardwareInterface</plugin>
+          <param name="CAN_CH">can0</param>
+        </hardware>
+      </xacro:if>
+      <!-- CAS 2 : GAZEBO SIMULATION -->
+      <xacro:unless value="${use_real_hardware}">
         <hardware>
           <plugin>gz_ros2_control/GazeboSimSystem</plugin>
         </hardware>
-      </xacro:if> -->
-      <!-- CAS 3 : VISUALISATION RViz (MOCK) -->
+      </xacro:unless>
+      <!-- CAS 3 : (MOCK) -->
       <!-- <xacro:unless value="${use_real_hardware or use_sim_time}">
         <hardware>
@@ -28,5 +27,5 @@
       </xacro:unless> -->
       <!-- ========================================================== -->
-      <!--            DÉFINITION DES ARTICULATIONS                    -->
+      <!--                    JOINTS DEFINITION                       -->
       <!-- ========================================================== -->
       <xacro:macro name="joint_definition" params="joint_name initial_pos">
@@ -39,5 +38,5 @@
         </joint>
       </xacro:macro>
-      <!-- On appelle la macro pour les 16 articulations -->
+      <!-- Call joint_definition macro for each joint -->
       <xacro:joint_definition joint_name="joint_00" initial_pos="joint_00" />
       <xacro:joint_definition joint_name="joint_01" initial_pos="joint_01" />
