Commit message: Update allegro_hand_description.urdf.xacro

File: allegro_hand_description/description/allegro_hand_description.urdf.xacro (robot description, xacro)
@@ -70,5 +70,5 @@
             <collision>
                 <geometry>
-                    <mesh filename="file://$(find allegro_hand_description)/meshes/hand/base_link_${suffix}_collision.stl"/>
+                    <mesh filename="file://$(find allegro_hand_description)/meshes/hand/base_link_${suffix}.stl"/>
                 </geometry>
             </collision>
@@ -97,5 +97,5 @@
                 <collision>
                     <geometry>
-                        <mesh filename="file://$(find allegro_hand_description)/meshes/hand/link_12_${suffix}_collision.stl"/>
+                        <mesh filename="file://$(find allegro_hand_description)/meshes/hand/link_12_${suffix}.stl"/>
                     </geometry>
                     <origin rpy="${zero_right * 180*DEG2RAD} 0 0" xyz="0 0 0"/>
@@ -131,5 +131,5 @@
                 <collision>
                     <geometry>
-                        <mesh filename="file://$(find allegro_hand_description)/meshes/hand/link_13_collision.stl"/>
+                        <mesh filename="file://$(find allegro_hand_description)/meshes/hand/link_13.stl"/>
                     </geometry>
                 </collision>
@@ -163,5 +163,5 @@
                 <collision>
                     <geometry>
-                        <mesh filename="file://$(find allegro_hand_description)/meshes/hand/link_14_collision.stl"/>
+                        <mesh filename="file://$(find allegro_hand_description)/meshes/hand/link_14.stl"/>
                     </geometry>
                 </collision>
@@ -195,5 +195,5 @@
                 <collision>
                     <geometry>
-                        <mesh filename="file://$(find allegro_hand_description)/meshes/hand/link_15_collision.stl"/>
+                        <mesh filename="file://$(find allegro_hand_description)/meshes/hand/link_15.stl"/>
                     </geometry>
                 </collision>
@@ -227,5 +227,5 @@
                 <collision>
                     <geometry>
-                        <mesh filename="file://$(find allegro_hand_description)/meshes/hand/link_15_tip_collision.stl"/>
+                        <mesh filename="file://$(find allegro_hand_description)/meshes/hand/link_15_tip.stl"/>
                     </geometry>
                 </collision>
@@ -260,5 +260,5 @@
                 <collision>
                     <geometry>
-                        <mesh filename="file://$(find allegro_hand_description)/meshes/hand/link_0_collision.stl"/>
+                        <mesh filename="file://$(find allegro_hand_description)/meshes/hand/link_0.stl"/>
                     </geometry>
                 </collision>
@@ -293,5 +293,5 @@
                 <collision>
                     <geometry>
-                        <mesh filename="file://$(find allegro_hand_description)/meshes/hand/link_1_collision.stl"/>
+                        <mesh filename="file://$(find allegro_hand_description)/meshes/hand/link_1.stl"/>
                     </geometry>
                 </collision>
@@ -325,5 +325,5 @@
                 <collision>
                     <geometry>
-                        <mesh filename="file://$(find allegro_hand_description)/meshes/hand/link_2_collision.stl"/>
+                        <mesh filename="file://$(find allegro_hand_description)/meshes/hand/link_2.stl"/>
                     </geometry>
                 </collision>
@@ -357,5 +357,5 @@
                 <collision>
                     <geometry>
-                        <mesh filename="file://$(find allegro_hand_description)/meshes/hand/link_3_collision.stl"/>
+                        <mesh filename="file://$(find allegro_hand_description)/meshes/hand/link_3.stl"/>
                     </geometry>
                 </collision>
@@ -389,5 +389,5 @@
                 <collision>
                     <geometry>
-                        <mesh filename="file://$(find allegro_hand_description)/meshes/hand/link_3_tip_collision.stl"/>
+                        <mesh filename="file://$(find allegro_hand_description)/meshes/hand/link_3_tip.stl"/>
                     </geometry>
                 </collision>
@@ -456,10 +456,10 @@
                 <collision>
                     <geometry>
-                        <mesh filename="file://$(find allegro_hand_description)/meshes/support/UR5_attachment_bottom_collision.stl" scale="0.001 0.001 0.001"/>
-                    </geometry>
-                </collision>
-                <collision>
-                    <geometry>
-                        <mesh filename="file://$(find allegro_hand_description)/meshes/support/UR5_attachment_top_collision.stl" scale="0.001 0.001 0.001"/>
+                        <mesh filename="file://$(find allegro_hand_description)/meshes/support/UR5_attachment_bottom.stl" scale="0.001 0.001 0.001"/>
+                    </geometry>
+                </collision>
+                <collision>
+                    <geometry>
+                        <mesh filename="file://$(find allegro_hand_description)/meshes/support/UR5_attachment_top.stl" scale="0.001 0.001 0.001"/>
                     </geometry>
                 </collision>
@@ -483,10 +483,10 @@
                 <collision>
                     <geometry>
-                        <mesh filename="file://$(find allegro_hand_description)/meshes/support/Allegro_deskstand_bottom_collision.stl" scale="0.001 0.001 0.001"/>
-                    </geometry>
-                </collision>
-                <collision>
-                    <geometry>
-                        <mesh filename="file://$(find allegro_hand_description)/meshes/support/Allegro_deskstand_top_collision.stl" scale="0.001 0.001 0.001"/>
+                        <mesh filename="file://$(find allegro_hand_description)/meshes/support/Allegro_deskstand_bottom.stl" scale="0.001 0.001 0.001"/>
+                    </geometry>
+                </collision>
+                <collision>
+                    <geometry>
+                        <mesh filename="file://$(find allegro_hand_description)/meshes/support/Allegro_deskstand_top.stl" scale="0.001 0.001 0.001"/>
                     </geometry>
                 </collision>
